File: QuadPassiveSwitch/quad_passive_switch.kicad_pcb (KiCad board)
At the start: 2 copper layers, 20 x 108.5 mm, 16 parts, among them J1 3.5mm_Mono_Switched_SymSmall_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, J10 3.5mm_Mono_Switched_SymSmall_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, J11 3.5mm_Mono_Switched_SymSmall_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, J12 3.5mm_Mono_Switched_SymSmall_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, J2 3.5mm_Mono_Switched_SymSmall_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, J3 3.5mm_Mono_Switched_SymSmall_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, J4 3.5mm_Mono_Switched_SymSmall_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, J5 3.5mm_Mono_Switched_SymSmall_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, J6 3.5mm_Mono_Switched_SymSmall_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, J7 3.5mm_Mono_Switched_SymSmall_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

Commit message: Add version to quad passive switch PCB
Other:
- board text added: "Oscen Quad Passive Switch, v1.0"
- board text added: "Quad Passive Switch"
- board text added: "v1.0"
